File: hardware/terminal_blocks.sch (KiCad schematic (older format))
At the start: 6 parts

Commit message: hardware: add TODOs in terminal_blocks
Other:
- note added: "TODO: move this to compartment light wire"
- note added: "TODO: switch this to AC for future?"
Changed lines of the file:
@@
 $Descr A4 11693 8268
 encoding utf-8
-Sheet 4 4
+Sheet 4 5
 Title ""
 Date ""
@@
 Text Notes 3990 3775 0    50   ~ 0
 Fridge Power
+Text Notes 4430 2345 0    50   ~ 0
+TODO: move this to compartment light wire
+Text Notes 4525 2485 0    50   ~ 0
+TODO: switch this to AC for future?
 $EndSCHEMATC

Commit message: hardware: add fuses to always on outputs
Parts:
- added F? (x8): 15A, symbol Device:Fuse
Connections:
- wire segments 36 -> 44
Other:
- note added: "TODO: add fuses"
Changed lines of the file:
@@
 	6555 4940 6555 4740
 Wire Wire Line
-	6730 4240 6490 4240
-Wire Wire Line
-	6730 4440 6490 4440
-Wire Wire Line
-	6730 4640 6490 4640
-Wire Wire Line
-	6730 4840 6490 4840
+	6100 4240 5860 4240
+Wire Wire Line
+	6100 4440 5860 4440
+Wire Wire Line
+	6100 4640 5860 4640
+Wire Wire Line
+	6100 4840 5860 4840
 Text HLabel 6455 2665 0    50   Input ~ 0
 AUX_SW_1
@@
 L power:+12V #PWR?
 U 1 1 60B4367C
-P 6490 4135
+P 5860 4135
 AR Path="/605C149A/60B4367C" Ref="#PWR?"  Part="1"
 AR Path="/60B2977E/60B4367C" Ref="#PWR?"  Part="1"
-F 0 "#PWR?" H 6490 3985 50  0001 C CNN
-F 1 "+12V" H 6505 4308 50  0000 C CNN
-F 2 "" H 6490 4135 50  0001 C CNN
-F 3 "" H 6490 4135 50  0001 C CNN
-	1    6490 4135
-	1    0    0    -1
-$EndComp
-Wire Wire Line
-	6490 4135 6490 4240
-Connection ~ 6490 4240
-Wire Wire Line
-	6490 4240 6490 4440
-Connection ~ 6490 4440
-Wire Wire Line
-	6490 4440 6490 4640
-Connection ~ 6490 4640
-Wire Wire Line
-	6490 4640 6490 4840
+F 0 "#PWR?" H 5860 3985 50  0001 C CNN
+F 1 "+12V" H 5875 4308 50  0000 C CNN
+F 2 "" H 5860 4135 50  0001 C CNN
+F 3 "" H 5860 4135 50  0001 C CNN
+	1    5860 4135
+	1    0    0    -1
+$EndComp
+Wire Wire Line
+	5860 4135 5860 4240
+Connection ~ 5860 4240
+Wire Wire Line
+	5860 4240 5860 4440
+Connection ~ 5860 4440
+Wire Wire Line
+	5860 4440 5860 4640
+Connection ~ 5860 4640
+Wire Wire Line
+	5860 4640 5860 4840
 Text Notes 6860 3990 0    50   ~ 0
 Always on AUX connections
@@
 Wire Wire Line
 	3675 1685 3740 1685
-Wire Wire Line
-	3740 1585 3675 1585
 $Comp
 L Connector_Generic:Conn_01x02 J?
@@
 Wire Wire Line
 	3675 2400 3740 2400
-Wire Wire Line
-	3740 2300 3675 2300
 $Comp
 L Connector_Generic:Conn_01x02 J?
@@
 Wire Wire Line
 	3670 3155 3735 3155
-Wire Wire Line
-	3735 3055 3670 3055
 $Comp
 L Connector_Generic:Conn_01x02 J?
@@
 	3670 3995 3735 3995
 Wire Wire Line
-	3735 3895 3670 3895
-$Comp
-L power:+12V #PWR?
-U 1 1 60B4F5A3
-P 3675 1585
-AR Path="/605C149A/60B4F5A3" Ref="#PWR?"  Part="1"
-AR Path="/60B2977E/60B4F5A3" Ref="#PWR?"  Part="1"
-F 0 "#PWR?" H 3675 1435 50  0001 C CNN
-F 1 "+12V" H 3690 1758 50  0000 C CNN
-F 2 "" H 3675 1585 50  0001 C CNN
-F 3 "" H 3675 1585 50  0001 C CNN
-	1    3675 1585
-	1    0    0    -1
-$EndComp
-$Comp
-L power:+12V #PWR?
-U 1 1 60B515C1
-P 3675 2300
-AR Path="/605C149A/60B515C1" Ref="#PWR?"  Part="1"
-AR Path="/60B2977E/60B515C1" Ref="#PWR?"  Part="1"
-F 0 "#PWR?" H 3675 2150 50  0001 C CNN
-F 1 "+12V" H 3690 2473 50  0000 C CNN
-F 2 "" H 3675 2300 50  0001 C CNN
-F 3 "" H 3675 2300 50  0001 C CNN
-	1    3675 2300
-	1    0    0    -1
-$EndComp
-$Comp
-L power:+12V #PWR?
-U 1 1 60B52355
-P 3670 3055
-AR Path="/605C149A/60B52355" Ref="#PWR?"  Part="1"
-AR Path="/60B2977E/60B52355" Ref="#PWR?"  Part="1"
-F 0 "#PWR?" H 3670 2905 50  0001 C CNN
-F 1 "+12V" H 3685 3228 50  0000 C CNN
-F 2 "" H 3670 3055 50  0001 C CNN
-F 3 "" H 3670 3055 50  0001 C CNN
-	1    3670 3055
-	1    0    0    -1
-$EndComp
+	3370 3895 3305 3895
 $Comp
 L power:+12V #PWR?
 U 1 1 60B5319F
-P 3670 3895
+P 3305 3895
 AR Path="/605C149A/60B5319F" Ref="#PWR?"  Part="1"
 AR Path="/60B2977E/60B5319F" Ref="#PWR?"  Part="1"
-F 0 "#PWR?" H 3670 3745 50  0001 C CNN
-F 1 "+12V" H 3685 4068 50  0000 C CNN
-F 2 "" H 3670 3895 50  0001 C CNN
-F 3 "" H 3670 3895 50  0001 C CNN
-	1    3670 3895
+F 0 "#PWR?" H 3305 3745 50  0001 C CNN
+F 1 "+12V" H 3320 4068 50  0000 C CNN
+F 2 "" H 3305 3895 50  0001 C CNN
+F 3 "" H 3305 3895 50  0001 C CNN
+	1    3305 3895
 	1    0    0    -1
 $EndComp
@@
 Text Notes 4525 2485 0    50   ~ 0
 TODO: switch this to AC for future?
+Text Notes 7155 4575 0    50   ~ 0
+TODO: add fuses
+$Comp
+L Device:Fuse F?
+U 1 1 606D8C52
+P 6250 4240
+F 0 "F?" V 6195 4085 50  0000 C CNN
+F 1 "15A" V 6330 4240 50  0000 C CNN
+F 2 "" V 6180 4240 50  0001 C CNN
+F 3 "~" H 6250 4240 50  0001 C CNN
+	1    6250 4240
+	0    1    1    0
+$EndComp
+$Comp
+L Device:Fuse F?
+U 1 1 606D98DE
+P 6250 4440
+F 0 "F?" V 6200 4285 50  0000 C CNN
+F 1 "15A" V 6325 4440 50  0000 C CNN
+F 2 "" V 6180 4440 50  0001 C CNN
+F 3 "~" H 6250 4440 50  0001 C CNN
+	1    6250 4440
+	0    1    1    0
+$EndComp
+$Comp
+L Device:Fuse F?
+U 1 1 606DA4A5
+P 6250 4640
+F 0 "F?" V 6200 4485 50  0000 C CNN
+F 1 "15A" V 6330 4640 50  0000 C CNN
+F 2 "" V 6180 4640 50  0001 C CNN
+F 3 "~" H 6250 4640 50  0001 C CNN
+	1    6250 4640
+	0    1    1    0
+$EndComp
+$Comp
+L Device:Fuse F?
+U 1 1 606DA997
+P 6250 4840
+F 0 "F?" V 6200 4685 50  0000 C CNN
+F 1 "15A" V 6330 4840 50  0000 C CNN
+F 2 "" V 6180 4840 50  0001 C CNN
+F 3 "~" H 6250 4840 50  0001 C CNN
+	1    6250 4840
+	0    1    1    0
+$EndComp
+Wire Wire Line
+	6730 4240 6400 4240
+Wire Wire Line
+	6730 4440 6400 4440
+Wire Wire Line
+	6730 4640 6400 4640
+Wire Wire Line
+	6730 4840 6400 4840
+$Comp
+L Device:Fuse F?
+U 1 1 606EDF10
+P 3520 3895
+F 0 "F?" V 3323 3895 50  0000 C CNN
+F 1 "15A" V 3414 3895 50  0000 C CNN
+F 2 "" V 3450 3895 50  0001 C CNN
+F 3 "~" H 3520 3895 50  0001 C CNN
+	1    3520 3895
+	0    1    1    0
+$EndComp
+Wire Wire Line
+	3735 3895 3670 3895
+Wire Wire Line
+	3370 3055 3305 3055
+$Comp
+L power:+12V #PWR?
+U 1 1 606FA025
+P 3305 3055
+AR Path="/605C149A/606FA025" Ref="#PWR?"  Part="1"
+AR Path="/60B2977E/606FA025" Ref="#PWR?"  Part="1"
+F 0 "#PWR?" H 3305 2905 50  0001 C CNN
+F 1 "+12V" H 3320 3228 50  0000 C CNN
+F 2 "" H 3305 3055 50  0001 C CNN
+F 3 "" H 3305 3055 50  0001 C CNN
+	1    3305 3055
+	1    0    0    -1
+$EndComp
+$Comp
+L Device:Fuse F?
+U 1 1 606FA02B
+P 3520 3055
+F 0 "F?" V 3323 3055 50  0000 C CNN
+F 1 "15A" V 3414 3055 50  0000 C CNN
+F 2 "" V 3450 3055 50  0001 C CNN
+F 3 "~" H 3520 3055 50  0001 C CNN
+	1    3520 3055
+	0    1    1    0
+$EndComp
+Wire Wire Line
+	3735 3055 3670 3055
+Wire Wire Line
+	3375 2300 3310 2300
+$Comp
+L power:+12V #PWR?
+U 1 1 606FB2CC
+P 3310 2300
+AR Path="/605C149A/606FB2CC" Ref="#PWR?"  Part="1"
+AR Path="/60B2977E/606FB2CC" Ref="#PWR?"  Part="1"
+F 0 "#PWR?" H 3310 2150 50  0001 C CNN
+F 1 "+12V" H 3325 2473 50  0000 C CNN
+F 2 "" H 3310 2300 50  0001 C CNN
+F 3 "" H 3310 2300 50  0001 C CNN
+	1    3310 2300
+	1    0    0    -1
+$EndComp
+$Comp
+L Device:Fuse F?
+U 1 1 606FB2D2
+P 3525 2300
+F 0 "F?" V 3328 2300 50  0000 C CNN
+F 1 "15A" V 3419 2300 50  0000 C CNN
+F 2 "" V 3455 2300 50  0001 C CNN
+F 3 "~" H 3525 2300 50  0001 C CNN
+	1    3525 2300
+	0    1    1    0
+$EndComp
+Wire Wire Line
+	3740 2300 3675 2300
+Wire Wire Line
+	3375 1585 3310 1585
+$Comp
+L power:+12V #PWR?
+U 1 1 606FC4BF
+P 3310 1585
+AR Path="/605C149A/606FC4BF" Ref="#PWR?"  Part="1"
+AR Path="/60B2977E/606FC4BF" Ref="#PWR?"  Part="1"
+F 0 "#PWR?" H 3310 1435 50  0001 C CNN
+F 1 "+12V" H 3325 1758 50  0000 C CNN
+F 2 "" H 3310 1585 50  0001 C CNN
+F 3 "" H 3310 1585 50  0001 C CNN
+	1    3310 1585
+	1    0    0    -1
+$EndComp
+$Comp
+L Device:Fuse F?
+U 1 1 606FC4C5
+P 3525 1585
+F 0 "F?" V 3328 1585 50  0000 C CNN
+F 1 "15A" V 3419 1585 50  0000 C CNN
+F 2 "" V 3455 1585 50  0001 C CNN
+F 3 "~" H 3525 1585 50  0001 C CNN
+	1    3525 1585
+	0    1    1    0
+$EndComp
+Wire Wire Line
+	3740 1585 3675 1585
 $EndSCHEMATC

Commit message: hardware: update comments
Other:
- note added: "OSTYK42102030"
- note added: "TODO: move this to compartment light wire. Replace with\n toilet power w/5A fuse?"
- note removed: "TODO: move this to compartment light wire"
- note removed: "TODO: switch this to AC for future?"
Changed lines of the file:
@@
 Fridge Power
 Text Notes 4430 2345 0    50   ~ 0
-TODO: move this to compartment light wire
-Text Notes 4525 2485 0    50   ~ 0
-TODO: switch this to AC for future?
+TODO: move this to compartment light wire. Replace with\n            toilet power w/5A fuse?
 Text Notes 7155 4575 0    50   ~ 0
 TODO: add fuses
@@
 Wire Wire Line
 	3740 1585 3675 1585
+Text Notes 4225 1675 0    50   ~ 0
+OSTYK42102030
 $EndSCHEMATC
