File: hardware/relays.sch (KiCad schematic (older format))
At the start: 100 parts

Commit message: hardware: remove diesel, fridge, and fan relays
Parts:
- removed D? (x4): D, Diode_SMD:D_SOD-123, symbol Device:D
- removed F? (x4): Fuse, symbol Device:Fuse
- removed K? (x4): DK1A-PS, switchboard:DK1A-PS, symbol switchboard:DK1A-PS
- removed Q? (x4): 2N7002, Package_TO_SOT_SMD:SOT-23, symbol Transistor_FET:2N7002
- removed R? (x4): 10K, Resistor_SMD:R_0805_2012Metric, symbol Device:R_US
Connections:
- net labels removed: DIESEL_HEATER, DIESEL_HEATER_CTRL, FRIDGE, FRIDGE_CTRL, KITCHEN_FAN, KITCHEN_FAN_CTRL, SHOWER_FAN, SHOWER_FAN_CTRL
- wire segments 400 -> 320
Other:
- moved on the sheet: R?

Commit message: hardware: add values for relay fuses
Parts:
- removed F? (x15): Fuse, symbol Device:Fuse
- added F? (x15): 7A, symbol Device:Fuse
- F?: value Fuse -> 7A
Changed lines of the file:
@@
 Text HLabel 2680 4130 2    50   Input ~ 0
 WATER_PUMP
-$Comp
-L Device:Fuse F?
-U 1 1 6084ED9D
-P 2530 4130
-F 0 "F?" V 2425 4130 50  0000 C CNN
-F 1 "Fuse" V 2424 4130 50  0001 C CNN
-F 2 "" V 2460 4130 50  0001 C CNN
-F 3 "~" H 2530 4130 50  0001 C CNN
-	1    2530 4130
-	0    1    1    0
-$EndComp
 Wire Wire Line
 	2310 3960 2350 3960
@@
 Wire Wire Line
 	2350 4130 2380 4130
-$Comp
-L Device:Fuse F?
-U 1 1 6088C7BD
-P 2530 2685
-F 0 "F?" V 2425 2685 50  0000 C CNN
-F 1 "Fuse" V 2424 2685 50  0001 C CNN
-F 2 "" V 2460 2685 50  0001 C CNN
-F 3 "~" H 2530 2685 50  0001 C CNN
-	1    2530 2685
-	0    1    1    0
-$EndComp
 Wire Wire Line
 	2310 2515 2350 2515
@@
 U 1 1 6089FDD9
 P 2530 5575
-F 0 "F?" V 2425 5575 50  0000 C CNN
-F 1 "Fuse" V 2424 5575 50  0001 C CNN
+F 0 "F?" V 2440 5575 50  0000 C CNN
+F 1 "7A" V 2615 5575 50  0000 C CNN
 F 2 "" V 2460 5575 50  0001 C CNN
 F 3 "~" H 2530 5575 50  0001 C CNN
@@
 Wire Wire Line
 	5040 1460 4780 1460
-$Comp
-L Device:Fuse F?
-U 1 1 6065CB49
-P 5715 5570
-F 0 "F?" V 5610 5570 50  0000 C CNN
-F 1 "Fuse" V 5609 5570 50  0001 C CNN
-F 2 "" V 5645 5570 50  0001 C CNN
-F 3 "~" H 5715 5570 50  0001 C CNN
-	1    5715 5570
-	0    1    1    0
-$EndComp
-$Comp
-L Device:Fuse F?
-U 1 1 6065CB4F
-P 5730 4125
-F 0 "F?" V 5625 4125 50  0000 C CNN
-F 1 "Fuse" V 5624 4125 50  0001 C CNN
-F 2 "" V 5660 4125 50  0001 C CNN
-F 3 "~" H 5730 4125 50  0001 C CNN
-	1    5730 4125
-	0    1    1    0
-$EndComp
 Wire Wire Line
 	5510 3955 5550 3955
@@
 Wire Wire Line
 	5525 5380 5510 5380
-$Comp
-L Device:Fuse F?
-U 1 1 6065CB5B
-P 5730 2680
-F 0 "F?" V 5625 2680 50  0000 C CNN
-F 1 "Fuse" V 5624 2680 50  0001 C CNN
-F 2 "" V 5660 2680 50  0001 C CNN
-F 3 "~" H 5730 2680 50  0001 C CNN
-	1    5730 2680
-	0    1    1    0
-$EndComp
 Wire Wire Line
 	5510 2510 5550 2510
@@
 Wire Wire Line
 	8485 1390 8225 1390
-$Comp
-L Device:Fuse F?
-U 1 1 607C5F7F
-P 9175 2610
-F 0 "F?" V 9070 2610 50  0000 C CNN
-F 1 "Fuse" V 9069 2610 50  0001 C CNN
-F 2 "" V 9105 2610 50  0001 C CNN
-F 3 "~" H 9175 2610 50  0001 C CNN
-	1    9175 2610
-	0    1    1    0
-$EndComp
 Wire Wire Line
 	8955 2440 8995 2440
@@
 Wire Wire Line
 	12690 8345 12730 8345
-$Comp
-L Device:Fuse F?
-U 1 1 607C5F88
-P 12910 8515
-F 0 "F?" V 12805 8515 50  0000 C CNN
-F 1 "Fuse" V 12804 8515 50  0001 C CNN
-F 2 "" V 12840 8515 50  0001 C CNN
-F 3 "~" H 12910 8515 50  0001 C CNN
-	1    12910 8515
-	0    1    1    0
-$EndComp
 Wire Wire Line
 	12830 7845 12690 7845
@@
 Wire Wire Line
 	12220 1395 11960 1395
-$Comp
-L Device:Fuse F?
-U 1 1 6092ED11
-P 12895 5505
-F 0 "F?" V 12790 5505 50  0000 C CNN
-F 1 "Fuse" V 12789 5505 50  0001 C CNN
-F 2 "" V 12825 5505 50  0001 C CNN
-F 3 "~" H 12895 5505 50  0001 C CNN
-	1    12895 5505
-	0    1    1    0
-$EndComp
-$Comp
-L Device:Fuse F?
-U 1 1 6092ED17
-P 12910 4060
-F 0 "F?" V 12805 4060 50  0000 C CNN
-F 1 "Fuse" V 12804 4060 50  0001 C CNN
-F 2 "" V 12840 4060 50  0001 C CNN
-F 3 "~" H 12910 4060 50  0001 C CNN
-	1    12910 4060
-	0    1    1    0
-$EndComp
 Wire Wire Line
 	12690 3890 12730 3890
@@
 Wire Wire Line
 	12705 5315 12690 5315
-$Comp
-L Device:Fuse F?
-U 1 1 6092ED23
-P 12910 2615
-F 0 "F?" V 12805 2615 50  0000 C CNN
-F 1 "Fuse" V 12804 2615 50  0001 C CNN
-F 2 "" V 12840 2615 50  0001 C CNN
-F 3 "~" H 12910 2615 50  0001 C CNN
-	1    12910 2615
-	0    1    1    0
-$EndComp
 Wire Wire Line
 	12690 2445 12730 2445
@@
 Wire Wire Line
 	12690 6830 12730 6830
-$Comp
-L Device:Fuse F?
-U 1 1 6092ED3E
-P 12910 7000
-F 0 "F?" V 12805 7000 50  0000 C CNN
-F 1 "Fuse" V 12804 7000 50  0001 C CNN
-F 2 "" V 12840 7000 50  0001 C CNN
-F 3 "~" H 12910 7000 50  0001 C CNN
-	1    12910 7000
-	0    1    1    0
-$EndComp
 Wire Wire Line
 	12830 6330 12690 6330
@@
 Wire Wire Line
 	9095 3385 8955 3385
-$Comp
-L Device:Fuse F?
-U 1 1 60713525
-P 9175 4055
-F 0 "F?" V 9070 4055 50  0000 C CNN
-F 1 "Fuse" V 9069 4055 50  0001 C CNN
-F 2 "" V 9105 4055 50  0001 C CNN
-F 3 "~" H 9175 4055 50  0001 C CNN
-	1    9175 4055
-	0    1    1    0
-$EndComp
 Wire Wire Line
 	8955 3885 8995 3885
@@
 Wire Wire Line
 	9095 4830 8955 4830
-$Comp
-L Device:Fuse F?
-U 1 1 60781D35
-P 9175 5500
-F 0 "F?" V 9070 5500 50  0000 C CNN
-F 1 "Fuse" V 9069 5500 50  0001 C CNN
-F 2 "" V 9105 5500 50  0001 C CNN
-F 3 "~" H 9175 5500 50  0001 C CNN
-	1    9175 5500
-	0    1    1    0
-$EndComp
 Wire Wire Line
 	8955 5330 8995 5330
@@
 Wire Wire Line
 	9095 6275 8955 6275
-$Comp
-L Device:Fuse F?
-U 1 1 607A33BA
-P 9175 6945
-F 0 "F?" V 9070 6945 50  0000 C CNN
-F 1 "Fuse" V 9069 6945 50  0001 C CNN
-F 2 "" V 9105 6945 50  0001 C CNN
-F 3 "~" H 9175 6945 50  0001 C CNN
-	1    9175 6945
-	0    1    1    0
-$EndComp
 Wire Wire Line
 	8955 6775 8995 6775
@@
 Wire Wire Line
 	9095 7720 8955 7720
-$Comp
-L Device:Fuse F?
-U 1 1 607D0BB4
-P 9175 8390
-F 0 "F?" V 9070 8390 50  0000 C CNN
-F 1 "Fuse" V 9069 8390 50  0001 C CNN
-F 2 "" V 9105 8390 50  0001 C CNN
-F 3 "~" H 9175 8390 50  0001 C CNN
-	1    9175 8390
-	0    1    1    0
-$EndComp
 Wire Wire Line
 	8955 8220 8995 8220
@@
 Connection ~ 8025 6675
 Connection ~ 8025 7720
+$Comp
+L Device:Fuse F?
+U 1 1 607D3D6A
+P 2530 4130
+F 0 "F?" V 2440 4130 50  0000 C CNN
+F 1 "7A" V 2615 4130 50  0000 C CNN
+F 2 "" V 2460 4130 50  0001 C CNN
+F 3 "~" H 2530 4130 50  0001 C CNN
+	1    2530 4130
+	0    1    1    0
+$EndComp
+$Comp
+L Device:Fuse F?
+U 1 1 607EFBFB
+P 2530 2685
+F 0 "F?" V 2440 2685 50  0000 C CNN
+F 1 "7A" V 2615 2685 50  0000 C CNN
+F 2 "" V 2460 2685 50  0001 C CNN
+F 3 "~" H 2530 2685 50  0001 C CNN
+	1    2530 2685
+	0    1    1    0
+$EndComp
+$Comp
+L Device:Fuse F?
+U 1 1 6080DE6F
+P 5730 2680
+F 0 "F?" V 5640 2680 50  0000 C CNN
+F 1 "7A" V 5815 2680 50  0000 C CNN
+F 2 "" V 5660 2680 50  0001 C CNN
+F 3 "~" H 5730 2680 50  0001 C CNN
+	1    5730 2680
+	0    1    1    0
+$EndComp
+$Comp
+L Device:Fuse F?
+U 1 1 60829D77
+P 5730 4125
+F 0 "F?" V 5640 4125 50  0000 C CNN
+F 1 "7A" V 5815 4125 50  0000 C CNN
+F 2 "" V 5660 4125 50  0001 C CNN
+F 3 "~" H 5730 4125 50  0001 C CNN
+	1    5730 4125
+	0    1    1    0
+$EndComp
+$Comp
+L Device:Fuse F?
+U 1 1 60847D78
+P 5715 5570
+F 0 "F?" V 5625 5570 50  0000 C CNN
+F 1 "7A" V 5800 5570 50  0000 C CNN
+F 2 "" V 5645 5570 50  0001 C CNN
+F 3 "~" H 5715 5570 50  0001 C CNN
+	1    5715 5570
+	0    1    1    0
+$EndComp
+$Comp
+L Device:Fuse F?
+U 1 1 6086B473
+P 9175 2610
+F 0 "F?" V 9085 2610 50  0000 C CNN
+F 1 "7A" V 9260 2610 50  0000 C CNN
+F 2 "" V 9105 2610 50  0001 C CNN
+F 3 "~" H 9175 2610 50  0001 C CNN
+	1    9175 2610
+	0    1    1    0
+$EndComp
+$Comp
+L Device:Fuse F?
+U 1 1 6088A3A6
+P 9175 4055
+F 0 "F?" V 9085 4055 50  0000 C CNN
+F 1 "7A" V 9260 4055 50  0000 C CNN
+F 2 "" V 9105 4055 50  0001 C CNN
+F 3 "~" H 9175 4055 50  0001 C CNN
+	1    9175 4055
+	0    1    1    0
+$EndComp
+$Comp
+L Device:Fuse F?
+U 1 1 608A887A
+P 9175 5500
+F 0 "F?" V 9085 5500 50  0000 C CNN
+F 1 "7A" V 9260 5500 50  0000 C CNN
+F 2 "" V 9105 5500 50  0001 C CNN
+F 3 "~" H 9175 5500 50  0001 C CNN
+	1    9175 5500
+	0    1    1    0
+$EndComp
+$Comp
+L Device:Fuse F?
+U 1 1 608C6FC4
+P 9175 6945
+F 0 "F?" V 9085 6945 50  0000 C CNN
+F 1 "7A" V 9260 6945 50  0000 C CNN
+F 2 "" V 9105 6945 50  0001 C CNN
+F 3 "~" H 9175 6945 50  0001 C CNN
+	1    9175 6945
+	0    1    1    0
+$EndComp
+$Comp
+L Device:Fuse F?
+U 1 1 608E2225
+P 9175 8390
+F 0 "F?" V 9085 8390 50  0000 C CNN
+F 1 "7A" V 9260 8390 50  0000 C CNN
+F 2 "" V 9105 8390 50  0001 C CNN
+F 3 "~" H 9175 8390 50  0001 C CNN
+	1    9175 8390
+	0    1    1    0
+$EndComp
+$Comp
+L Device:Fuse F?
+U 1 1 608FEA33
+P 12910 8515
+F 0 "F?" V 12820 8515 50  0000 C CNN
+F 1 "7A" V 12995 8515 50  0000 C CNN
+F 2 "" V 12840 8515 50  0001 C CNN
+F 3 "~" H 12910 8515 50  0001 C CNN
+	1    12910 8515
+	0    1    1    0
+$EndComp
+$Comp
+L Device:Fuse F?
+U 1 1 6091CC84
+P 12910 7000
+F 0 "F?" V 12820 7000 50  0000 C CNN
+F 1 "7A" V 12995 7000 50  0000 C CNN
+F 2 "" V 12840 7000 50  0001 C CNN
+F 3 "~" H 12910 7000 50  0001 C CNN
+	1    12910 7000
+	0    1    1    0
+$EndComp
+$Comp
+L Device:Fuse F?
+U 1 1 6093C5E4
+P 12895 5505
+F 0 "F?" V 12805 5505 50  0000 C CNN
+F 1 "7A" V 12980 5505 50  0000 C CNN
+F 2 "" V 12825 5505 50  0001 C CNN
+F 3 "~" H 12895 5505 50  0001 C CNN
+	1    12895 5505
+	0    1    1    0
+$EndComp
+$Comp
+L Device:Fuse F?
+U 1 1 609585B3
+P 12910 4060
+F 0 "F?" V 12820 4060 50  0000 C CNN
+F 1 "7A" V 12995 4060 50  0000 C CNN
+F 2 "" V 12840 4060 50  0001 C CNN
+F 3 "~" H 12910 4060 50  0001 C CNN
+	1    12910 4060
+	0    1    1    0
+$EndComp
+$Comp
+L Device:Fuse F?
+U 1 1 6097679B
+P 12910 2615
+F 0 "F?" V 12820 2615 50  0000 C CNN
+F 1 "7A" V 12995 2615 50  0000 C CNN
+F 2 "" V 12840 2615 50  0001 C CNN
+F 3 "~" H 12910 2615 50  0001 C CNN
+	1    12910 2615
+	0    1    1    0
+$EndComp
 $EndSCHEMATC

Commit message: hardware: migrate to VN750 instead of relays
Parts:
- removed D? (x16): D, Diode_SMD:D_SOD-123, symbol Device:D
- removed F? (x16): 7A, symbol Device:Fuse
- removed K? (x16): DK1A-PS, switchboard:DK1A-PS, symbol switchboard:DK1A-PS
- removed Q? (x16): 2N7002, Package_TO_SOT_SMD:SOT-23, symbol Transistor_FET:2N7002
- removed R? (x16): 10K, Resistor_SMD:R_0805_2012Metric, symbol Device:R_US
- added C?: 0.33uF, Capacitor_SMD:C_0805_2012Metric_Pad1.18x1.45mm_HandSolder, symbol Device:C
- added C?: 0.1uF, Capacitor_SMD:C_0805_2012Metric_Pad1.18x1.45mm_HandSolder, symbol Device:C
- added R? (x24): 10k, Resistor_SMD:R_0805_2012Metric_Pad1.20x1.40mm_HandSolder, symbol Device:R_US
- added R? (x24): 2k, Resistor_SMD:R_0805_2012Metric_Pad1.20x1.40mm_HandSolder, symbol Device:R_US
- added U? (x24): TCMT4600, Package_SO:SOP-16_4.55x10.3mm_P1.27mm, symbol switchboard:VN750
- added U? (x24): TCMT4600, Package_SO:SOP-16_4.55x10.3mm_P1.27mm, symbol Isolator:TCMT4600
- added U?: TCMT4600, Package_SO:SOP-16_4.55x10.3mm_P1.27mm, symbol Regulator_Linear:L7805
Connections:
- net labels added: +12V_house, +5V, AUX_1_CTRL_12V, AUX_1_OUT0, AUX_1_OUT1, AUX_1_OUT[0..1], AUX_2_CTRL_12V, AUX_2_OUT0, AUX_2_OUT1, AUX_2_OUT[0..1], AUX_3_CTRL_12V, AUX_3_OUT0, AUX_3_OUT1, AUX_3_OUT[0..1], AUX_4_CTRL_12V, AUX_4_OUT0, AUX_4_OUT1, AUX_4_OUT[0..1], BAR_LIGHT0, BAR_LIGHT1, BAR_LIGHT[0..1], BAR_LIGHT_CTRL_12V, BENCH_DOME_A0, BENCH_DOME_A1, BENCH_DOME_A[0..1], BENCH_DOME_B0, BENCH_DOME_B1, BENCH_DOME_B[0..1], COMP_1_CTRL_12V, COMP_1_LIGHT0, COMP_1_LIGHT1, COMP_1_LIGHT[0..1], COMP_2_CTRL_12V, COMP_2_LIGHT0, COMP_2_LIGHT1, COMP_2_LIGHT[0..1], COMP_3_CTRL_12V, COMP_3_LIGHT0, COMP_3_LIGHT1, COMP_3_LIGHT[0..1], COMP_4_CTRL_12V, COMP_4_LIGHT0, COMP_4_LIGHT1, COMP_4_LIGHT[0..1], COMP_5_CTRL_12V, COMP_5_LIGHT0, COMP_5_LIGHT1, COMP_5_LIGHT[0..1], COT_DOME_A0, COT_DOME_A1, COT_DOME_A[0..1], COT_DOME_B0, COT_DOME_B1, COT_DOME_B[0..1], DOME_CTRL_12V, DRIVER_FLOOD_A0, DRIVER_FLOOD_A1, DRIVER_FLOOD_A[0..1], DRIVER_FLOOD_B0, DRIVER_FLOOD_B1, DRIVER_FLOOD_B[0..1], DRIVER_FLOOD_CTRL_12V, PASS_FLOOD_A0, PASS_FLOOD_A1, PASS_FLOOD_A[0..1], PASS_FLOOD_B0, PASS_FLOOD_B1, PASS_FLOOD_B[0..1], PASS_FLOOD_CTRL_12V, REAR_FLOOD_A0, REAR_FLOOD_A1, REAR_FLOOD_A[0..1], REAR_FLOOD_B0, REAR_FLOOD_B1, REAR_FLOOD_B[0..1], REAR_FLOOD_CTRL_12V, STRIP_LIGHT_C0, STRIP_LIGHT_C1, STRIP_LIGHT_CTRL_12V, STRIP_LIGHT_C[0..1], STRIP_LIGHT_F0, STRIP_LIGHT_F1, STRIP_LIGHT_F[0..1], STRIP_LIGHT_R0, STRIP_LIGHT_R1, STRIP_LIGHT_R[0..1], WATER_PUMP0, WATER_PUMP1, WATER_PUMP[0..1], WATER_PUMP_CTRL_12V
- net labels removed: +12V, AUX_RLY_1, AUX_RLY_1_CTRL, AUX_RLY_2, AUX_RLY_2_CTRL, AUX_RLY_3, AUX_RLY_3_CTRL, AUX_RLY_4, AUX_RLY_4_CTRL, BAR_LIGHT, BAR_LIGHT_CTRL, COMP_1_LIGHT, COMP_1_LIGHT_CTRL, COMP_2_LIGHT, COMP_2_LIGHT_CTRL, COMP_3_LIGHT, COMP_3_LIGHT_CTRL, COMP_4_LIGHT, COMP_4_LIGHT_CTRL, COMP_5_LIGHT, COMP_5_LIGHT_CTRL, DOME_LIGHTS, DOME_LIGHTS_CTRL, DRIVER_FLOOD, DRIVER_FLOOD_CTRL, PASS_FLOOD, PASS_FLOOD_CTRL, REAR_FLOOD, REAR_FLOOD_CTRL, STRIP_LIGHTS, STRIP_LIGHTS_CTRL, WATER_PUMP, WATER_PUMP_CTRL
- wire segments 320 -> 397
- no-connect marks 0 -> 24
Other:
- note added: "Compartment Lights"
- note added: "Flood Lights"
- note added: "Interior Components"
- note added: "Interior Lights"
