File: hardware/relays.sch (KiCad schematic (older format))
At the start: 99 parts

Commit message: hardware: add truck high-side drivers
Parts:
- added R? (x26): 10k, Resistor_SMD:R_0805_2012Metric_Pad1.20x1.40mm_HandSolder, symbol Device:R_US
- added R? (x26): 2k, Resistor_SMD:R_0805_2012Metric_Pad1.20x1.40mm_HandSolder, symbol Device:R_US
- added U? (x26): TCMT4600, Package_SO:SOP-16_4.55x10.3mm_P1.27mm, symbol Isolator:TCMT4600
- added U? (x26): TCMT4600, Package_SO:SOP-16_4.55x10.3mm_P1.27mm, symbol switchboard:VN750
Connections:
- net +5V: now also U?.16, U?.16, U?.16, U?.16, U?.16, U?.16, U?.16, U?.16, U?.16, U?.16, U?.16, U?.16, U?.16, U?.16, U?.16, U?.16, U?.16, U?.16, U?.16, U?.16, U?.16, U?.16, U?.16, U?.16, U?.16, U?.16
- net GNDREF: now also R?.1, R?.1, R?.1, R?.1, R?.1, R?.1, R?.1, R?.1, R?.1, R?.1, R?.1, R?.1, R?.1, R?.1, R?.1, R?.1, R?.1, R?.1, R?.1, R?.1, R?.1, R?.1, R?.1, R?.1, R?.1, R?.1, R?.1, R?.1, R?.1, R?.1, R?.1, R?.1, R?.1, R?.1, R?.1, R?.1, R?.1, R?.1, R?.1, R?.1, R?.1, R?.1, R?.1, R?.1, R?.1, R?.1, R?.1, R?.1, R?.1, R?.1, R?.1, R?.1, U?.1 (GND), U?.1 (GND), U?.1 (GND), U?.1 (GND), U?.1 (GND), U?.1 (GND), U?.1 (GND), U?.1 (GND), U?.1 (GND), U?.1 (GND), U?.1 (GND), U?.1 (GND), U?.1 (GND), U?.1 (GND), U?.1 (GND), U?.1 (GND), U?.1 (GND), U?.1 (GND), U?.1 (GND), U?.1 (GND), U?.1 (GND), U?.1 (GND), U?.1 (GND), U?.1 (GND), U?.1 (GND), U?.1 (GND)
- new net: R?.2, U?.15, U?.2 (x26)
- new net: R?.2, U?.2 (x26)
- new net BACKUP_ALARM0: U?.3
- new net BACKUP_ALARM1: U?.5
- new net BACKUP_ALARM_CTRL_12V: U?.1
- new net CURB_FRONT_RED0: U?.3
- new net CURB_FRONT_RED1: U?.5
- new net CURB_FRONT_RED_CTRL_12V: U?.1
- new net CURB_REAR_RED0: U?.3
- new net CURB_REAR_RED1: U?.5
- new net CURB_REAR_RED_CTRL_12V: U?.1
- new net FOG_CTRL_12V: U?.1, U?.1
- new net FOG_CURB0: U?.3
- new net FOG_CURB1: U?.5
- new net FOG_STREET0: U?.3
- new net FOG_STREET1: U?.5
- new net GRILLE_STROBE0: U?.3
- new net GRILLE_STROBE1: U?.5
- new net GRILLE_STROBE_CTRL_12V: U?.1
- new net HEADLAMP_HI_L0: U?.3
- new net HEADLAMP_HI_L1: U?.5
- new net HEADLAMP_HI_L_CTRL_12V: U?.1
- new net HEADLAMP_HI_R0: U?.3
- new net HEADLAMP_HI_R1: U?.5
- new net HEADLAMP_HI_R_CTRL_12V: U?.1
- new net LIGHT_BAR_A0: U?.3
- new net LIGHT_BAR_A1: U?.5
- new net LIGHT_BAR_A_CTRL_12V: U?.1
- new net LIGHT_BAR_B0: U?.3
- new net LIGHT_BAR_B1: U?.5
- new net LIGHT_BAR_B_CTRL_12V: U?.1
- new net LIGHT_BAR_C0: U?.3
- new net LIGHT_BAR_C1: U?.5
- new net LIGHT_BAR_C_CTRL_12V: U?.1
- new net LIGHT_BAR_D0: U?.3
- new net LIGHT_BAR_D1: U?.5
- new net LIGHT_BAR_D_CTRL_12V: U?.1
- new net LIGHT_BAR_E0: U?.3
- new net LIGHT_BAR_E1: U?.5
- new net LIGHT_BAR_E_CTRL_12V: U?.1
- new net LIGHT_BAR_F0: U?.3
- new net LIGHT_BAR_F1: U?.5
- new net LIGHT_BAR_F_CTRL_12V: U?.1
- new net LIGHT_BAR_G0: U?.3
- new net LIGHT_BAR_G1: U?.5
- new net LIGHT_BAR_G_CTRL_12V: U?.1
- new net MARKER_CTRL_12V: U?.1, U?.1
- new net MARKER_LIGHTS_A0: U?.3
- new net MARKER_LIGHTS_A1: U?.5
- new net MARKER_LIGHTS_B0: U?.3
- new net MARKER_LIGHTS_B1: U?.5
- new net PACK_POWER_A0: U?.3
- new net PACK_POWER_A1: U?.5
- new net PACK_POWER_B0: U?.3
- new net PACK_POWER_B1: U?.5
- new net PACK_POWER_CTRL_12V: U?.1, U?.1
- new net REAR_LOW_CURB0: U?.3
- new net REAR_LOW_CURB1: U?.5
- new net REAR_LOW_CURB_CTRL_12V: U?.1
- new net REAR_LOW_STREET0: U?.3
- new net REAR_LOW_STREET1: U?.5
- new net REAR_LOW_STREET_CTRL_12V: U?.1
- new net REAR_STROBE0: U?.3
- new net REAR_STROBE1: U?.5
- new net REAR_STROBE_CTRL_12V: U?.1
- new net SECURITY_RELAY0: U?.3
- new net SECURITY_RELAY1: U?.5
- new net SECURITY_RELAY_CTRL_12V: U?.1
- new net STREET_FRONT_RED0: U?.3
- new net STREET_FRONT_RED1: U?.5
- new net STREET_FRONT_RED_CTRL_12V: U?.1
- new net STREET_REAR_RED0: U?.3
- new net STREET_REAR_RED1: U?.5
- new net STREET_REAR_RED_CTRL_12V: U?.1
- new net STROBE_PATTERN0: U?.3
- new net STROBE_PATTERN1: U?.5
- new net STROBE_PATTERN_CTRL_12V: U?.1
- no-connect marks 24 -> 50
Other:
- note added: "Flasher Components"
- note added: "House Battery"
- note added: "Truck Battery"
- note added: "Truck Components"
- moved on the sheet: C?, U?
